Commit message: Update mobile_base.urdf

File: ROS_Files/src/mobile_robot/mobile_base/mobile_base.urdf (robot description, URDF)
Before this commit: robot two_wheeled_robot, 4 links, 3 joints
Links:
- link back_caster: geometry collision sphere radius=${(wheel_radius+wheel_zoff-(base_height/2))}
- link front_caster: geometry collision sphere radius=${(wheel_radius+wheel_zoff-(base_height/2))}
