Commit message: Update arm_base.urdf.xacro

File: ROS_Files/src/mobile_robot/arm_base.urdf.xacro (robot description, xacro)
@@ -2,13 +2,16 @@
 <robot xmlns:xacro="http://ros.org/wiki/xacro" name="mobile_manipulator" >
 <!-- base-->
-<xacro:include filename="$(find robot_body)/urdf/mobile_base/mobile_base.urdf" />
-<xacro:include filename="$(find robot_body)/urdf/ur5e/ur5e_macro.xacro" />
-<xacro:ur5e_robot prefix="ur5e_"/>
-<gazebo>
-  <plugin filename="libgazebo_ros2_control.so" name="gazebo_ros2_control">
-    <parameters>$(find robot_body)/config/robot_controllers.yaml</parameters>
-  </plugin>
-</gazebo>
-<!-- Attacher link between arm and base-->
+<xacro:include filename="$(find mobile_base)/urdf/mobile_base/basic_mobile_bot_v2.urdf" />
+<!-- ur5e-->
+  <!-- Arm model -->
+  <xacro:include filename="$(find mobile_base)/urdf/ur5e/ur5e_macro.xacro" />
+  <xacro:ur5e_robot prefix="ur5e_"/>
+  <!-- Gazebo control plugin for the arm -->
+   <gazebo>
+    <plugin filename="libgazebo_ros2_control.so" name="gazebo_ros2_control">
+      <parameters>$(find mobile_base)/config/robot_controllers.yaml</parameters>
+    </plugin>
+  </gazebo>
+<!-- Create a box to attach arm to -->
 <link name="box_link">
     <visual>
@@ -29,5 +32,5 @@
 </link>
 <gazebo reference="box_link">
-    <material>Gazebo/Purple</material>
+    <material>Gazebo/Pioneer2Body</material>
   </gazebo>
 <joint name="box_joint" type="fixed">
@@ -36,9 +39,10 @@
     <origin xyz="0 0 0.15" rpy="0 0 0"/>
 </joint>
-<joint name="box_ur5e" type="fixed">
-  <parent link="box_link"/>
-  <child link="ur5e_base_link"/>
-  <origin xyz="0.0 0.0 0.0" rpy="0 0 0"/>
-</joint>
+<!-- Connect Arm to Base -->
+  <joint name="box_ur5e" type="fixed">
+    <parent link="box_link"/>
+    <child link="ur5e_base_link"/>
+    <origin xyz="0.0 0.0 0.0" rpy="0 0 0"/>
+  </joint>
 <!-- Include robotiq_2f_85 gripper -->
  <xacro:include filename="$(find robotiq_description)/urdf/robotiq_2f_85_macro.urdf.xacro" />
@@ -148,3 +152,22 @@
     <origin xyz="0.0 0.0 0.1603" rpy="0 0 0"/>
 </joint>
+<!--
+ <material name="blue">
+    <color rgba="0 0 0.8 1"/>
+  </material>
+<link name="box_link">
+    <visual>
+	<origin rpy="0 0 0" xyz="0 0 0"/>
+      <geometry>
+        <box size="0.75 0.45 0.49"/>
+      </geometry>
+	<material name="blue"/>
+    </visual>
+</link>
+<joint name="box_mir100" type="fixed">
+    <parent link="surface"/>
+    <child link="box_link"/>
+    <origin xyz="0 0 0.245" rpy="0 0 0"/>
+</joint>
+-->
 </robot>
